Commit message: polish hopper mpc example

File: examples/models/hopper.urdf (robot description, URDF)
Before this commit: robot hopper, 3 links, 3 joints
Links:
- link torso: geometry collision capsule length=0.4 radius=.05; visual capsule length=0.4 radius=.05

Commit message: remove non-sphere collision geometry from hopper

File: examples/models/hopper.urdf (robot description, URDF)
Before this commit: robot hopper, 3 links, 3 joints
Links:
- link torso: geometry visual capsule length=0.4 radius=.05
